Commit message: 20210213

File: opdracht2/urdf/opdracht2a.xacro (robot description, xacro)
@@ -6,7 +6,13 @@
   <xacro:include filename="$(find toets_support)/urdf/workshop/workshop.urdf.xacro"/>
   <xacro:workshop_urdf workshop_parent="world_interface"/>
+  <!-- Joints -->
+  <joint name="world_interface_to_world" type="fixed">
+    <parent link="world" />
+    <child link="world_interface" />
+    <origin xyz="1 0 0.0" rpy="0 0 0"/>
+  </joint>
   <!-- hall -->
   <xacro:include filename="$(find toets_support)/urdf/hall/hall.urdf.xacro"/>
-  <xacro:hall_urdf hall_parent="world"  hall_prefix="hall_" >
+  <xacro:hall_urdf hall_parent="world_interface"  hall_prefix="hall_" >
     <origin xyz="-2.5 0 0.0" rpy="0 0 0"/>
   </xacro:hall_urdf>
@@ -25,14 +31,14 @@
   <xacro:include filename="$(find toets_support)/urdf/bin/bin.urdf.xacro"/>
   <xacro:bin_urdf prefix="bin_1_"/>
-  <!-- Joints -->
-  <joint name="world_interface_to_world" type="fixed">
-    <parent link="world" />
-    <child link="world_interface" />
-  </joint>
   <!-- robot1-pedestal to world. -->
   <joint name="robot1_pedestal_to_world_interface" type="fixed">
+<!--
     <parent link="world_interface" />
     <child link="robot1_pedestal_link" />
     <origin xyz="-4 0 0.0" rpy="0 0.0 0.0"/>
+-->
+    <parent link="world" />
+    <child link="robot1_pedestal_link" />
+    <origin xyz="0 0 0.0" rpy="0 0.0 0.0"/>
   </joint>
   <!-- robot1 to pedestal. -->

Commit message: 20210218

File: opdracht2/urdf/opdracht2a.xacro (robot description, xacro)
@@ -10,5 +10,5 @@
     <parent link="world" />
     <child link="world_interface" />
-    <origin xyz="1 0 0.0" rpy="0 0 0"/>
+    <origin xyz="0 0 0.0" rpy="0 0 0"/>
   </joint>
   <!-- hall -->
@@ -17,4 +17,9 @@
     <origin xyz="-2.5 0 0.0" rpy="0 0 0"/>
   </xacro:hall_urdf>
+  <!-- pallet -->
+  <xacro:include filename="$(find toets_support)/urdf/pallet/pallet.urdf.xacro"/>
+  <xacro:pallet_urdf pallet_parent="world_interface" pallet_prefix="pallet_">
+    <origin xyz="-5 2 0.0" rpy="0 0 0"/>
+  </xacro:pallet_urdf>
   <!-- Robot1 Pedestal -->
   <xacro:include filename="$(find toets_support)/urdf/robot_pedestal/robot_pedestal.urdf.xacro"/>
@@ -33,12 +38,7 @@
   <!-- robot1-pedestal to world. -->
   <joint name="robot1_pedestal_to_world_interface" type="fixed">
-<!--
-    <parent link="world_interface" />
+    <parent link="world" />
     <child link="robot1_pedestal_link" />
     <origin xyz="-4 0 0.0" rpy="0 0.0 0.0"/>
--->
-    <parent link="world" />
-    <child link="robot1_pedestal_link" />
-    <origin xyz="0 0 0.0" rpy="0 0.0 0.0"/>
   </joint>
   <!-- robot1 to pedestal. -->

File: toets_support/urdf/toets.xacro (robot description, xacro)
@@ -9,5 +9,5 @@
   <xacro:include filename="$(find toets_support)/urdf/hall/hall.urdf.xacro"/>
   <xacro:hall_urdf hall_prefix="hall_" hall_parent="world_interface">
-    <origin xyz="2.5 0 0.0" rpy="0 0 0"/>
+    <origin xyz="-2.5 0 0.0" rpy="0 0 0"/>
   </xacro:hall_urdf>
   <!-- Robot1 Pedestal -->
@@ -35,27 +35,8 @@
     <child link="world_interface" />
   </joint>
-  <!-- robot1-pedestal to world. -->
-<!--
-  <joint name="robot1_pedestal_to_world_interface" type="fixed">
-    <parent link="world_interface" />
-    <child link="robot1_pedestal_link" />
-    <origin xyz="4 0 0.0" rpy="0.0 0.0 0.0"/>
-  </joint>
--->
-  <!-- hall-pedestal to world. -->
-<!--
-  <joint name="hall_to_world_interface" type="fixed">
-    <parent link="world_interface" />
-    <child link="hall_link" />
-    <origin xyz="0 0 0.0" rpy="0.0 0.0 0.0"/>
-  </joint>
--->
   <!-- robot1 to pedestal. -->
   <joint name="robot1_to_pedestal" type="fixed">
-  <origin xyz="0 0 0.95" rpy="0 0 1.57" />
+  <origin xyz="0 0 0.95" rpy="0 0 -1.57" />
     <parent link="robot1_pedestal_link" />
-<!--
-  <parent link="world_interface" />
--->
   <child link="robot1_base_link" />
   </joint>

File: toets_support/urdf/vacuum_gripper/vacuum_gripper.urdf.xacro (robot description, xacro)
@@ -55,8 +55,11 @@
     <!-- joint list -->
     <joint name="${joint_prefix}" type="fixed">
-      <origin xyz="0 0 0.01" rpy="0 0 0" />
+      <origin xyz="0 0 0.08" rpy="0 0 0" />
       <parent link="${prefix}base_link" />
       <child link="${prefix}suction_cup" />
     </joint>
+  <gazebo reference="${prefix}suction_cup">
+    <material>Gazebo/Red</material>
+  </gazebo>
   </xacro:macro>
 </robot>
