Commit message: 20210221-3

File: opdracht2/urdf/environment1.xacro (robot description, xacro)
@@ -17,9 +17,4 @@
     <origin xyz="-2.5 0 0.0" rpy="0 0 0"/>
   </xacro:hall_urdf>
-  <!-- pallet -->
-  <xacro:include filename="$(find toets_support)/urdf/pallet/pallet.urdf.xacro"/>
-  <xacro:pallet_urdf pallet_parent="world_interface" pallet_prefix="pallet_">
-    <origin xyz="-5 2 0.0" rpy="0 0 0"/>
-  </xacro:pallet_urdf>
   <!-- Robot1 Pedestal -->
   <xacro:include filename="$(find toets_support)/urdf/robot_pedestal/robot_pedestal.urdf.xacro"/>

File: toets_support/urdf/pallet/pallet.urdf.xacro (robot description, xacro)
@@ -8,5 +8,5 @@
   </joint>
     <!-- Links -->
-<link name="${pallet_parent}"/>
+    <link name="${pallet_parent}"/>
     <link name="${pallet_prefix}origin">
       <visual>
