Commit message: 20210302

File: casus_support/urdf/hall/hall.urdf.xacro (robot description, xacro)
@@ -23,5 +23,5 @@
     <child link="${hall_prefix}floor"/>
   </joint>
-	<xacro:property name="dummy_thickness" value="0.001" />
+	<xacro:property name="dummy_thickness" value="0.01" />
 	<xacro:property name="dummy_mass" value="100" />
   <material name="${hall_prefix}floor_color">
@@ -38,5 +38,5 @@
 			<geometry>
 			 <box size="${depth} ${width} ${dummy_thickness}"/>
-	        <origin xyz="1 1. -1" rpy="0 0 0" />
+	        <origin xyz="0 0 -${dummy_thickness}" rpy="0 0 0" />
 			</geometry>
 			<material name="${hall_prefix}floor_color"/>
