Commit message: 20210509

File: casus_support/urdf/casus.xacro (robot description, xacro)
@@ -3,15 +3,25 @@
   <!-- world -->
   <link name="world" />
+  <!-- world to world_interface. -->
+  <joint name="world_to_world_interface" type="fixed">
+    <parent link="world" />
+    <child link="world_interface" />
+  </joint>
   <!-- workcell -->
   <xacro:include filename="$(find casus_support)/urdf/workshop/workshop.urdf.xacro"/>
-  <xacro:workshop_urdf workshop_parent="world_interface"/>
+  <xacro:workshop_urdf workshop_parent="world"/>
   <!-- hall -->
   <xacro:include filename="$(find casus_support)/urdf/hall/hall.urdf.xacro"/>
-  <xacro:hall_urdf hall_prefix="hall_" hall_parent="world_interface">
+  <xacro:hall_urdf hall_prefix="hall_" hall_parent="world">
     <origin xyz="-2.5 0 0.0" rpy="0 0 0"/>
   </xacro:hall_urdf>
+  <!-- Mobile Computer -->
+  <xacro:include filename="$(find casus_support)/urdf/computer_mobile/computer.urdf.xacro"/>
+  <xacro:computer_urdf computer_parent="world" computer_prefix="comp_mobile_" >
+  <origin xyz="-5 0 0" rpy="0 0 2.1"/>
+  </xacro:computer_urdf>
   <!-- Robot1 Pedestal -->
   <xacro:include filename="$(find casus_support)/urdf/robot_pedestal/robot_pedestal.urdf.xacro"/>
-  <xacro:robot_pedestal_urdf pedestal_prefix="robot1_" pedestal_parent="world_interface" pedestal_height="0.95">
+  <xacro:robot_pedestal_urdf pedestal_prefix="robot1_" pedestal_parent="world" pedestal_height="0.95">
     <origin xyz="-4 -1 0.0" rpy="0 0 0"/>
   </xacro:robot_pedestal_urdf>
@@ -25,14 +35,4 @@
   <xacro:include filename="$(find casus_support)/urdf/bin/bin.urdf.xacro"/>
   <xacro:bin_urdf prefix="bin_1_"/>
-  <!-- logical camera 1 collision model -->
-  <xacro:include filename="$(find casus_support)/urdf/logical_camera/logical_camera.urdf.xacro"/>
-  <xacro:logical_camera_urdf prefix="logical_camera1_" logical_camera_parent="world_interface">
-    <origin xyz="-3 -0.4 1.75" rpy="0 1.5708 0"/>
-  </xacro:logical_camera_urdf>
-  <!-- Joints -->
-  <joint name="world_interface_to_world" type="fixed">
-    <parent link="world" />
-    <child link="world_interface" />
-  </joint>
   <!-- robot1 to pedestal. -->
   <joint name="robot1_to_pedestal" type="fixed">
@@ -48,5 +48,5 @@
   <!-- bin to world. -->
   <joint name="bin_1_joint" type="fixed">
-    <parent link="world_interface" />
+    <parent link="world" />
     <child link="bin_1_base_link" />
     <origin xyz="-4 -2 0.0" rpy="0 0 0" />

File: casus_support/urdf/forklift/forklift.urdf.xacro (robot description, xacro)
@@ -8,5 +8,7 @@
   </joint>
     <!-- Links -->
+<!--
 <link name="${forklift_parent}"/>
+-->
     <link name="${forklift_prefix}origin">
       <visual>

File: casus_support/urdf/hall/hall.urdf.xacro (robot description, xacro)
@@ -23,8 +23,8 @@
     <child link="${hall_prefix}floor"/>
   </joint>
-	<xacro:property name="dummy_thickness" value="0.01" />
-	<xacro:property name="dummy_mass" value="100" />
+    <xacro:property name="dummy_thickness" value="0.01" />
+    <xacro:property name="dummy_mass" value="100" />
   <material name="${hall_prefix}floor_color">
-	<color rgba="${0/255} ${255/255} ${0/255} 1"/>
+    <color rgba="${0/255} ${255/255} ${0/255} 1"/>
   </material>
   <material name="${hall_prefix}wall1_color">
@@ -34,120 +34,120 @@
     <color rgba="${255/255} ${255/255} ${0/255} 1"/>
   </material>
-	<link name="${hall_prefix}floor">
-		<visual>
-			<geometry>
-			 <box size="${depth} ${width} ${dummy_thickness}"/>
-	        <origin xyz="0 0 -${dummy_thickness}" rpy="0 0 0" />
-			</geometry>
-			<material name="${hall_prefix}floor_color"/>
-		</visual>
+    <link name="${hall_prefix}floor">
+        <visual>
+            <geometry>
+             <box size="${depth} ${width} ${dummy_thickness}"/>
+            <origin xyz="0 0 -${dummy_thickness}" rpy="0 0 0" />
+            </geometry>
+            <material name="${hall_prefix}floor_color"/>
+        </visual>
       <collision>
-			<geometry>
-			 <box size="${depth} ${width} ${dummy_thickness}"/>
-	        <origin xyz="0 0 -0.1" rpy="0 0 0" />
-			</geometry>
+            <geometry>
+             <box size="${depth} ${width} ${dummy_thickness}"/>
+            <origin xyz="0 0 -0.1" rpy="0 0 0" />
+            </geometry>
       </collision>
       <inertial>
         <origin xyz="0 0 0" rpy="0 0 0" />
-		<xacro:box_inertia m="${dummy_mass}" x="${depth}" y="${width}" z="${dummy_thickness}"/>
+        <xacro:box_inertia m="${dummy_mass}" x="${depth}" y="${width}" z="${dummy_thickness}"/>
         <mass value="${dummy_mass}" />
       </inertial>
-	</link>
-	<link name="${hall_prefix}wall1">
-		<visual>
-			<geometry>
-			 <box size="${depth} ${height} ${dummy_thickness}"/>
-			</geometry>
-			<origin rpy="0 0 0" xyz="0 0 -${dummy_thickness}"/>
-			<material name="${hall_prefix}wall1_color"/>
-		</visual>
+    </link>
+    <link name="${hall_prefix}wall1">
+        <visual>
+            <geometry>
+             <box size="${depth} ${height} ${dummy_thickness}"/>
+            </geometry>
+            <origin rpy="0 0 0" xyz="0 0 -${dummy_thickness}"/>
+            <material name="${hall_prefix}wall1_color"/>
+        </visual>
       <collision>
-			<geometry>
-			 <box size="${depth} ${height} ${dummy_thickness}"/>
-			</geometry>
+            <geometry>
+             <box size="${depth} ${height} ${dummy_thickness}"/>
+            </geometry>
       </collision>
       <inertial>
         <origin xyz="0 0 0" rpy="0 0 0" />
-		<xacro:box_inertia m="${dummy_mass}" x="${depth}" y="${height}" z="${dummy_thickness}"/>
+        <xacro:box_inertia m="${dummy_mass}" x="${depth}" y="${height}" z="${dummy_thickness}"/>
         <mass value="${dummy_mass}" />
       </inertial>
-	</link>
-	<joint name="${hall_prefix}floor_to_wall1" type="fixed">
-		<parent link="${hall_prefix}floor"/>
-		<child link="${hall_prefix}wall1"/>
-		<origin rpy="1.56 0 0" xyz="0 ${0.5 * width} ${0.5 * height}"/>
-	</joint>
-	<link name="${hall_prefix}wall2">
-		<visual>
-			<geometry>
-			 <box size="${height} ${width} ${dummy_thickness}"/>
-			</geometry>
-			<origin rpy="0 0 0" xyz="0 0 -${dummy_thickness}"/>
-			<material name="${hall_prefix}wall2_color"/>
-		</visual>
+    </link>
+    <joint name="${hall_prefix}floor_to_wall1" type="fixed">
+        <parent link="${hall_prefix}floor"/>
+        <child link="${hall_prefix}wall1"/>
+        <origin rpy="1.56 0 0" xyz="0 ${0.5 * width} ${0.5 * height}"/>
+    </joint>
+    <link name="${hall_prefix}wall2">
+        <visual>
+            <geometry>
+             <box size="${height} ${width} ${dummy_thickness}"/>
+            </geometry>
+            <origin rpy="0 0 0" xyz="0 0 -${dummy_thickness}"/>
+            <material name="${hall_prefix}wall2_color"/>
+        </visual>
       <collision>
-			<geometry>
-			 <box size="${height} ${width} ${dummy_thickness}"/>
-			</geometry>
+            <geometry>
+             <box size="${height} ${width} ${dummy_thickness}"/>
+            </geometry>
       </collision>
       <inertial>
         <origin xyz="0 0 0" rpy="0 0 0" />
-		<xacro:box_inertia m="${dummy_mass}" x="${height}" y="${width}" z="${dummy_thickness}"/>
+        <xacro:box_inertia m="${dummy_mass}" x="${height}" y="${width}" z="${dummy_thickness}"/>
         <mass value="${dummy_mass}" />
       </inertial>
-	</link>
-	<joint name="${hall_prefix}floor_to_wall2" type="fixed">
-		<parent link="${hall_prefix}floor"/>
-		<child link="${hall_prefix}wall2"/>
-		<origin rpy="0 1.56 0" xyz="${0.5 * depth} 0 ${0.5 * height}"/>
-	</joint>
-	<link name="${hall_prefix}wall3">
-		<visual>
-			<geometry>
-			 <box size="${depth} 0.5 ${dummy_thickness}"/>
-			</geometry>
-			<origin rpy="0 0 0" xyz="0 0 -${dummy_thickness}"/>
-			<material name="${hall_prefix}wall1_color"/>
-		</visual>
+    </link>
+    <joint name="${hall_prefix}floor_to_wall2" type="fixed">
+        <parent link="${hall_prefix}floor"/>
+        <child link="${hall_prefix}wall2"/>
+        <origin rpy="0 1.56 0" xyz="${0.5 * depth} 0 ${0.5 * height}"/>
+    </joint>
+    <link name="${hall_prefix}wall3">
+        <visual>
+            <geometry>
+             <box size="${depth} 0.5 ${dummy_thickness}"/>
+            </geometry>
+            <origin rpy="0 0 0" xyz="0 0 -${dummy_thickness}"/>
+            <material name="${hall_prefix}wall1_color"/>
+        </visual>
       <collision>
-			<geometry>
-			 <box size="${depth} 0.5 ${dummy_thickness}"/>
-			</geometry>
+            <geometry>
+             <box size="${depth} 0.5 ${dummy_thickness}"/>
+            </geometry>
       </collision>
       <inertial>
         <origin xyz="0 0 0" rpy="0 0 0" />
-		<xacro:box_inertia m="${dummy_mass}" x="${depth}" y="0.5" z="${dummy_thickness}"/>
+        <xacro:box_inertia m="${dummy_mass}" x="${depth}" y="0.5" z="${dummy_thickness}"/>
         <mass value="${dummy_mass}" />
       </inertial>
-	</link>
-	<joint name="${hall_prefix}world_interface_to_wall3" type="fixed">
-		<parent link="${hall_prefix}floor"/>
-		<child link="${hall_prefix}wall3"/>
-		<origin rpy="1.56 0 0" xyz="0 -${0.5 * width} ${0.5 * 0.5}"/>
-	</joint>
-	<link name="${hall_prefix}wall4">
-		<visual>
-			<geometry>
-			 <box size="0.5 ${width} ${dummy_thickness}"/>
-			</geometry>
-			<origin rpy="0 0 0" xyz="0 0 -${dummy_thickness}"/>
-			<material name="${hall_prefix}wall2_color"/>
-		</visual>
+    </link>
+    <joint name="${hall_prefix}world_interface_to_wall3" type="fixed">
+        <parent link="${hall_prefix}floor"/>
+        <child link="${hall_prefix}wall3"/>
+        <origin rpy="1.56 0 0" xyz="0 -${0.5 * width} ${0.5 * 0.5}"/>
+    </joint>
+    <link name="${hall_prefix}wall4">
+        <visual>
+            <geometry>
+             <box size="0.5 ${width} ${dummy_thickness}"/>
+            </geometry>
+            <origin rpy="0 0 0" xyz="0 0 -${dummy_thickness}"/>
+            <material name="${hall_prefix}wall2_color"/>
+        </visual>
       <collision>
-			<geometry>
-			 <box size="0.5 ${width} ${dummy_thickness}"/>
-			</geometry>
+            <geometry>
+             <box size="0.5 ${width} ${dummy_thickness}"/>
+            </geometry>
       </collision>
       <inertial>
         <origin xyz="0 0 0" rpy="0 0 0" />
-		<xacro:box_inertia m="${dummy_mass}" x="0.5" y="${width}" z="${dummy_thickness}"/>
+        <xacro:box_inertia m="${dummy_mass}" x="0.5" y="${width}" z="${dummy_thickness}"/>
         <mass value="${dummy_mass}" />
       </inertial>
-	</link>
-	<joint name="${hall_prefix}world_interface_to_wall4" type="fixed">
-		<parent link="${hall_prefix}floor"/>
-		<child link="${hall_prefix}wall4"/>
-		<origin rpy="0 1.56 0" xyz="-${0.5 * depth} 0 ${0.5 * 0.5}"/>
-	</joint>
+    </link>
+    <joint name="${hall_prefix}world_interface_to_wall4" type="fixed">
+        <parent link="${hall_prefix}floor"/>
+        <child link="${hall_prefix}wall4"/>
+        <origin rpy="0 1.56 0" xyz="-${0.5 * depth} 0 ${0.5 * 0.5}"/>
+    </joint>
   <gazebo reference="${hall_prefix}floor">
     <material>Gazebo/Green</material>

File: casus_support/urdf/hall/hall.xacro (robot description, xacro)
@@ -8,9 +8,13 @@
   <xacro:arg name="x" default="0"/>
   <xacro:arg name="y" default="0"/>
+  <xacro:arg name="z" default="0"/>
+  <xacro:arg name="R" default="0"/>
+  <xacro:arg name="P" default="0"/>
+  <xacro:arg name="Y" default="0"/>
   <!-- URDF -->
   <link name="world_interface"/>
   <xacro:include filename="$(find casus_support)/urdf/hall/hall.urdf.xacro"/>
   <xacro:hall_urdf hall_prefix="$(arg hall_prefix)" hall_parent="$(arg hall_parent)" width ="$(arg width)" depth ="$(arg depth)" height ="$(arg height)">
-    <origin xyz="$(arg x) $(arg y) 0" rpy="0 0 0"/>
+     <origin xyz="$(arg x) $(arg y) $(arg z)" rpy="$(arg R) $(arg P) $(arg Y)"/>
   </xacro:hall_urdf>
 </robot>

File: casus_support/urdf/logical_camera/logical_camera.urdf.xacro (robot description, xacro)
@@ -6,7 +6,7 @@
     <xacro:property name="height" value="0.050"/>
     <joint name="${prefix}logical_camera_joint" type="fixed">
-	<xacro:insert_block name="origin" />
-	<parent link="${logical_camera_parent}"/>
-	<child link="${prefix}base_link"/>
+    <xacro:insert_block name="origin" />
+    <parent link="${logical_camera_parent}"/>
+    <child link="${prefix}base_link"/>
     </joint>
     <!-- link list -->

File: casus_support/urdf/pallet/pallet.urdf.xacro (robot description, xacro)
@@ -8,5 +8,7 @@
   </joint>
     <!-- Links -->
+<!--
     <link name="${pallet_parent}"/>
+-->
     <link name="${pallet_prefix}origin">
       <visual>

File: casus_support/urdf/pallettruck/pallettruck.urdf.xacro (robot description, xacro)
@@ -8,5 +8,7 @@
   </joint>
     <!-- Links -->
+<!--
 <link name="${pallettruck_parent}"/>
+-->
     <link name="${pallettruck_prefix}origin">
       <visual>

File: casus_support/urdf/robot_pedestal/robot_pedestal.urdf.xacro (robot description, xacro)
@@ -1,36 +1,36 @@
 <?xml version="1.0" ?>
 <robot name="robot_pedestal_urdf" xmlns:xacro="http://www.ros.org/wiki/xacro">
-<!-- robot pedestal -->
-<xacro:macro name = "robot_pedestal_urdf" params = "pedestal_prefix pedestal_parent pedestal_height *origin">
-  <joint name="${pedestal_prefix}pedestal_joint" type="fixed">
+    <!-- robot pedestal -->
+    <xacro:macro name = "robot_pedestal_urdf" params = "pedestal_prefix pedestal_parent pedestal_height *origin">
+    <joint name="${pedestal_prefix}pedestal_joint" type="fixed">
     <xacro:insert_block name="origin" />
     <parent link="${pedestal_parent}"/>
     <child link="${pedestal_prefix}pedestal_link"/>
-  </joint>
-  <link name="${pedestal_prefix}pedestal_link">
-    <visual>
-      <origin xyz="0 0 ${0.5*pedestal_height}"/>
-      <geometry>
-        <box size="0.3 0.3 ${pedestal_height}"/>
-      </geometry>
-      <material name="pedestal_color">
-        <color rgba="0 ${40/255} ${134/255} 1"/>
-      </material>
-    </visual>
-    <collision>
-      <origin xyz="0 0 ${0.5*pedestal_height}"/>
-      <geometry>
-        <box size="0.3 0.3 ${pedestal_height}"/>
-      </geometry>
-    </collision>
-    <inertial>
-      <mass value="500"/>
-      <origin xyz="0 0 0" rpy="0 0 0"/>
-      <inertia ixx="0.001" ixy="0" ixz="0" iyy="0.001" iyz="0" izz="0.001"/>
-    </inertial>
-  </link>
-  <gazebo reference="${pedestal_prefix}pedestal_link">
-    <material>Gazebo/Blue</material>
-  </gazebo>
-</xacro:macro>
+    </joint>
+    <link name="${pedestal_prefix}pedestal_link">
+        <visual>
+            <origin xyz="0 0 ${0.5*pedestal_height}"/>
+            <geometry>
+            <box size="0.3 0.3 ${pedestal_height}"/>
+            </geometry>
+            <material name="pedestal_color">
+            <color rgba="0 ${40/255} ${134/255} 1"/>
+            </material>
+        </visual>
+        <collision>
+            <origin xyz="0 0 ${0.5*pedestal_height}"/>
+            <geometry>
+            <box size="0.3 0.3 ${pedestal_height}"/>
+            </geometry>
+        </collision>
+        <inertial>
+            <mass value="500"/>
+            <origin xyz="0 0 0" rpy="0 0 0"/>
+            <inertia ixx="0.001" ixy="0" ixz="0" iyy="0.001" iyz="0" izz="0.001"/>
+            </inertial>
+    </link>
+    <gazebo reference="${pedestal_prefix}pedestal_link">
+        <material>Gazebo/Blue</material>
+    </gazebo>
+    </xacro:macro>
 </robot>

File: casus_support/urdf/workshop/workshop.urdf.xacro (robot description, xacro)
@@ -2,6 +2,6 @@
 <robot name="workshop_urdf" xmlns:xacro="http://www.ros.org/wiki/xacro">
     <xacro:macro name="workshop_urdf" params="workshop_parent">
+    <link name="world_interface"/>
     <!-- Links -->
-    <link name="world_interface"/>
     <link name="workshop">
       <visual>
