Commit message: 20210510

File: casus2/urdf/environment.xacro (robot description, xacro)
@@ -3,4 +3,9 @@
   <!-- world -->
   <link name="world" />
+   <!-- world to world_interface. -->
+  <joint name="world_to_world_interface" type="fixed">
+    <parent link="world" />
+    <child link="world_interface" />
+  </joint>
   <!-- workshop -->
   <xacro:include filename="$(find casus_support)/urdf/workshop/workshop.urdf.xacro"/>

File: casus2/urdf/uitwerking.xacro (robot description, xacro)
@@ -3,4 +3,9 @@
     <!-- world -->
     <link name="world" />
+   <!-- world to world_interface. -->
+  <joint name="world_to_world_interface" type="fixed">
+    <parent link="world" />
+    <child link="world_interface" />
+  </joint>
   <!-- workshop -->
   <xacro:include filename="$(find casus_support)/urdf/workshop/workshop.urdf.xacro"/>
